File: _autosave-RadProt_IOT.kicad_pcb (KiCad board)
At the start: 2 copper layers, 76 x 55 mm, 10 parts, among them J1 Conn_01x04_Pin, J2 Conn_01x04_Pin, J3 Conn_01x04_Pin, J6 Conn_02x05_Top_Bottom, SW1 Config, U1 RaspberryPi_Pico_W

Commit message: gcode generated...
Parts:
- moved D1 12.6 mm to (108.1, 113.1)
- moved R1 9.91 mm to (108.1, 126.6), turned to 90 degrees
- moved SW1 2.90 mm to (111.9, 124.6), turned to 0 degrees
- renumbered J6 to J1, J1 to UART1, J2 to UART2, J3 to UART3
Routing:
- net Net-(U1-GPIO15): track 7.23 -> 19.1 mm
- net Net-(U1-GPIO14): track 19.7 -> 12.4 mm
- net Net-(D1-A): track 3.40 -> 5.89 mm
- net GND: track 108.0 -> 110.3 mm
- net Net-(U1-GPIO19): track 43.5 -> 41.5 mm
- net Net-(U1-GPIO18): track 32.6 -> 33.5 mm
Other:
- outline, holes or cut-outs redrawn
