File: RadProt_IOT.kicad_pcb (KiCad board)
At the start: 2 copper layers, 76 x 55 mm, 10 parts, among them J1 Conn_01x04_Pin, J2 Conn_01x04_Pin, J3 Conn_01x04_Pin, J6 Conn_02x05_Top_Bottom, SW1 Config, U1 RaspberryPi_Pico_W

Commit message: gcode generated...
Parts:
- moved D1 12.6 mm to (108.1, 113.1)
- moved R1 9.91 mm to (108.1, 126.6), turned to 90 degrees
- moved SW1 2.90 mm to (111.9, 124.6), turned to 0 degrees
- renumbered J6 to J1, J1 to UART1, J2 to UART2, J3 to UART3
Routing:
- net Net-(U1-GPIO15): track 7.23 -> 19.1 mm
- net Net-(U1-GPIO14): track 19.7 -> 12.4 mm
- net +5V: track 80.1 -> 74.6 mm
- net Net-(D1-A): track 3.40 -> 5.89 mm
- net Net-(U1-GPIO16): track 46.8 -> 49.2 mm
- net GND: track 108.0 -> 110.3 mm
- net Net-(U1-GPIO20): track 35.7 -> 37.9 mm
- net Net-(U1-GPIO21): track 43.6 -> 42.0 mm
- net Net-(U1-GPIO18): track 33.0 -> 33.5 mm
- added copper zone on B.Cu, net +5V
Other:
- outline, holes or cut-outs redrawn

Commit message: prepared univprepared universal board with this layout
Parts:
- removed UART1: Conn_01x04_Pin, Connector_PinHeader_2.54mm:PinHeader_1x04_P2.54mm_Vertical
- added UART0: Conn_01x04_Socket, Connector_PinSocket_2.54mm:PinSocket_1x04_P2.54mm_Vertical, F.Cu at (107.0, 91.3)
- R1: footprint Resistor_THT:R_Axial_DIN0204_L3.6mm_D1.6mm_P5.08mm_Horizontal -> Resistor_THT:R_Axial_DIN0204_L3.6mm_D1.6mm_P7.62mm_Horizontal
- UART2, UART3: value Conn_01x04_Pin -> Conn_01x04_Socket; footprint Connector_PinHeader_2.54mm:PinHeader_1x04_P2.54mm_Vertical -> Connector_PinSocket_2.54mm:PinSocket_1x04_P2.54mm_Vertical
- moved UART3 57.3 mm to (107.0, 157.1), turned to 180 degrees
- moved UART2 34.9 mm to (107.0, 124.1), turned to 180 degrees
- moved R1 13.7 mm to (117.1, 116.3), turned to -90 degrees
- moved D1 9.06 mm to (117.1, 113.9), turned to 90 degrees
- moved GND 8.45 mm to (115.2, 100.5)
- moved +5V 8.26 mm to (115.2, 95.4)
- moved SW1 2.88 mm to (114.0, 126.6)
- moved ENC28J60 0.26 mm to (166.8, 126.7)
- renumbered +5v to +5V, J1 to ENC28J60
Connections:
- D1 pad 1: GND -> Net-(D1-K)
- R1 pad 1: Net-(U1-GPIO15) -> Net-(D1-K)
- R1 pad 2: Net-(D1-A) -> GND
- SW1 pad 2: Net-(U1-GPIO14) -> Net-(U1-GPIO15)
- U1 pad 12: unconnected-(U1-GPIO9-Pad12) -> Net-(D1-A)
- U1 pad 19: Net-(U1-GPIO14) -> unconnected-(U1-GPIO14-Pad19)
- UART2 pad 3: (no net) -> unconnected-(UART2-Pin_3-Pad3)
- UART3 pad 3: (no net) -> unconnected-(UART3-Pin_3-Pad3)
Routing:
- net +5V: track 74.6 -> 148.2 mm
- net /UART3_RX: track 13.5 -> 65.0 mm
- net /UART2_RX: track 5.97 -> 41.3 mm
- net GND: track 110.3 -> 78.7 mm, vias 0 -> 2
- net Net-(U1-GPIO14): track 12.4 -> 0.00 mm
- net Net-(U1-GPIO15): track 19.1 -> 11.0 mm
- net /UART0_RX: track 12.5 -> 19.1 mm
- net Net-(U1-GPIO16): track 49.2 -> 52.5 mm
- net Net-(U1-GPIO20): track 37.9 -> 35.2 mm
- net Net-(U1-GPIO18): track 33.5 -> 36.1 mm
- net Net-(D1-K): track 0.00 -> 2.40 mm
- net Net-(D1-A): track 5.89 -> 7.08 mm
- removed copper zone on B.Cu, net +5V
Other:
- board size 76 x 55 mm -> 80 x 80 mm
- board text removed: "TX"
