File: MAX3232_Module.kicad_block/MAX3232_Module.kicad_sch (KiCad schematic)
At the start: 1 part, among them J1 Conn_01x04_Pin

Commit message: prepared univprepared universal board with this layout
Parts:
- removed J1: Conn_01x04_Pin, symbol Connector:Conn_01x04_Pin
- added J1: Conn_01x04_Socket, symbol Connector:Conn_01x04_Socket
Changed lines of the file:
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@@
 	(paper "A4")
 	(image
-		(at 148.59 101.6)
-		(scale 0.686556)
+		(at 147.32 101.854)
+		(scale 0.646691)
 		(data "iVBORw0KGgoAAAANSUhEUgAAAr8AAAK6CAYAAAAw1DRdAAAABHNCSVQICAgIfAhkiAAAAAlwSFlz"
 			"AAAuGAAALhgBKqonIAAAIABJREFUeJzsvWusbV2a1/V7xhhzznXbZ59z3kvVe6kquhs6sdEYCQLG"
@@
 	)
 	(symbol
-		(lib_id "Connector:Conn_01x04_Pin")
-		(at 166.37 100.33 0)
+		(lib_id "Connector:Conn_01x04_Socket")
+		(at 163.83 100.33 0)
+		(mirror y)
 		(unit 1)
 		(exclude_from_sim no)
@@
 		(fields_autoplaced yes)
 		(property "Reference" "J1"
-			(at 167.005 92.71 0)
+			(at 164.465 92.71 0)
 			(effects
 				(font
@@
 			)
 		)
-		(property "Value" "Conn_01x04_Pin"
-			(at 167.005 95.25 0)
+		(property "Value" "Conn_01x04_Socket"
+			(at 164.465 95.25 0)
 			(effects
 				(font
 					(size 1.27 1.27)
 				)
-				(hide yes)
 			)
 		)
 		(property "Footprint" ""
-			(at 166.37 100.33 0)
+			(at 163.83 100.33 0)
 			(effects
 				(font
@@
 		)
 		(property "Datasheet" "~"
-			(at 166.37 100.33 0)
+			(at 163.83 100.33 0)
 			(effects
 				(font
@@
 		)
 		(property "Description" "Generic connector, single row, 01x04, script generated"
-			(at 166.37 100.33 0)
+			(at 163.83 100.33 0)
 			(effects
 				(font
@@
 		(pin "2"
 		)
-		(pin "4"
-		)
 		(pin "1"
 		)
+		(pin "4"
+		)
 		(instances
